File: ADC.kicad_sch (KiCad schematic)
At the start: 0 parts

Commit message: All done, Gerberd out :)
Parts:
- added C38, C39, C40, C42: 0.1uF, Capacitor_SMD:C_0603_1608Metric, symbol majed-symbols:C
- added C41: 10uF 25V 1206, Capacitor_SMD:C_1206_3216Metric, symbol majed-symbols:C
- added R33: 100K, Resistor_SMD:R_0603_1608Metric, symbol majed-symbols:R_Small_US
- added R34: 0, Resistor_SMD:R_0603_1608Metric, symbol majed-symbols:R_Small_US
- added R35: DNI, Resistor_SMD:R_0603_1608Metric, symbol majed-symbols:R_Small_US
- added TP11: SCK, TestPoint:TestPoint_Pad_1.0x1.0mm, symbol majed-symbols:TestPoint
- added TP12: BUSY, TestPoint:TestPoint_Pad_1.0x1.0mm, symbol majed-symbols:TestPoint
- added TP13: MOSI, TestPoint:TestPoint_Pad_1.0x1.0mm, symbol majed-symbols:TestPoint
- added TP14: CNV, TestPoint:TestPoint_Pad_1.0x1.0mm, symbol majed-symbols:TestPoint
- added TP15: /CS, TestPoint:TestPoint_Pad_1.0x1.0mm, symbol majed-symbols:TestPoint
- added TP16: REF, TestPoint:TestPoint_Pad_1.0x1.0mm, symbol majed-symbols:TestPoint
- added U10: AD4630-24, Majed-footprints:05-08-1797_ADI-L, symbol majed-symbols:AD4630-ADC
Connections:
- new net: C41.1, C42.1, R34.1, U10.A2 (REFIN)
- new net +1.8V: C38.1, C39.1, R33.1, U10.A8 (VIO), U10.B8 (VIO), U10.G3 (VDD_1.8V), U10.H3 (VDD_1.8V)
- new net +5V: C40.1, U10.A3 (VDD_5V), U10.B3 (VDD_5V)
- new net BUSY: TP12.1, U10.E8 (BUSY)
- new net CNV: TP14.1, U10.A6 (CNV)
- new net GND: C38.2, C39.2, C40.2, C41.2, C42.2, U10.A1 (GND), U10.A4 (GND), U10.A5 (GND), U10.B2 (GND), U10.B4 (GND), U10.B5 (GND), U10.B6 (IOGND), U10.B7 (IOGND), U10.C2 (GND), U10.C3 (GND), U10.C4 (GND), U10.C5 (GND), U10.C6 (IOGND), U10.D1 (GND), U10.D4 (GND), U10.D5 (GND), U10.D6 (IOGND), U10.E1 (GND), U10.E4 (GND), U10.E5 (GND), U10.E6 (IOGND), U10.E7 (IOGND), U10.F2 (GND), U10.F3 (GND), U10.F4 (GND), U10.F5 (GND), U10.F6 (IOGND), U10.G2 (GND), U10.G4 (GND), U10.G5 (GND), U10.G6 (IOGND), U10.H1 (GND), U10.H2 (GND), U10.H4 (GND), U10.H8 (IOGND)
- new net IN_A+: U10.B1 (IN0+)
- new net IN_A-: U10.C1 (IN0-)
- new net IN_B+: U10.F1 (IN1+)
- new net IN_B-: U10.G1 (IN1-)
- new net MISO0: U10.D8 (SDO0)
- new net MOSI: TP13.1, U10.H6 (SDI)
- new net REF: R35.2, TP16.1, U10.D2 (REF), U10.D3 (REF), U10.E2 (REF), U10.E3 (REF)
- new net REF_5V: R34.2, R35.1
- new net SCK: TP11.1, U10.H7 (SCK)
- new net /CS: TP15.1, U10.H5 (CS*)
- new net /RESET: R33.2, U10.A7 (RESET*)
- no-connect marks 0 -> 7
Other:
- note added: "Analog Interface"
- note added: "Power and Reference"
