File: MCU-FPGA.kicad_sch (KiCad schematic)
At the start: 0 parts

Commit message: All done, Gerberd out :)
Parts:
- added C25, C28, C29, C30, C31, C32, C33, C34, C35, C36, C37: 0.1uF, Capacitor_SMD:C_0603_1608Metric, symbol majed-symbols:C_Small
- added C26, C27: 4.7uF, Capacitor_SMD:C_0805_2012Metric, symbol majed-symbols:C_Small
- added D13: LED_RGB, Majed-footprints:APHF1608SEEQBDZGKC_KNB-L, symbol majed-symbols:LED_APHF1608SEEQBDZGKC
- added FB7: 33R, Inductor_SMD:L_0603_1608Metric_Pad1.05x0.95mm_HandSolder, symbol majed-symbols:FerriteBead
- added J7: STM32 PROGRAMER, Majed-footprints:SPARKFUN_PRT-14417, symbol majed-symbols:STM_PROGRAMER_PRT-14417
- added J8: USB_B_Micro, Connector_USB:USB_Micro-B_Molex-105017-0001, symbol majed-symbols:USB_B_Micro-Connector_1
- added Q1: 2N7002K, Package_TO_SOT_SMD:SOT-23, symbol majed-symbols:2N7002K
- added R23, R24: 400, Resistor_SMD:R_0603_1608Metric, symbol majed-symbols:R_Small_US
- added R25: 825, Resistor_SMD:R_0603_1608Metric, symbol majed-symbols:R_Small_US
- added R26, R29, R30, R31, R32: 10K, Resistor_SMD:R_0603_1608Metric, symbol majed-symbols:R_Small_US
- added R27: 100, Resistor_SMD:R_0603_1608Metric, symbol majed-symbols:R_Small_US
- added R28: 20K, Resistor_SMD:R_0603_1608Metric, symbol majed-symbols:R_Small_US
- added SW1: Push - BOOT, Button_Switch_SMD:SW_Tactile_SPST_NO_Straight_CK_PTS636Sx25SMTRLFS, symbol majed-symbols:SW_Push
- added TP10: GND, TestPoint:TestPoint_Pad_1.0x1.0mm, symbol majed-symbols:TestPoint
- added TP7: UART4_RX, TestPoint:TestPoint_Pad_1.0x1.0mm, symbol majed-symbols:TestPoint
- added TP8: UART4_TX, TestPoint:TestPoint_Pad_1.0x1.0mm, symbol majed-symbols:TestPoint
- added TP9: UART4_CTS, TestPoint:TestPoint_Pad_1.0x1.0mm, symbol majed-symbols:TestPoint
- added U7: STM32H730VBT6, Package_QFP:LQFP-100_14x14mm_P0.5mm, symbol majed-symbols:STM32H730VBTx
- added U8: ESDA6V1BC6, Package_TO_SOT_SMD:SOT-23-6, symbol majed-symbols:ESDA6V1BC6
- added U9: ECS-1612MV-120-CN-TR, Majed-footprints:ECS-1612MV-120-CN-TR, symbol majed-symbols:ECS-1612MV-120-CN-TR
Connections:
- new net: C25.1, FB7.2, U7.20 (VREF+)
- new net: J8.1 (VBUS), R31.1
- new net: C26.1, U7.48 (VCAP)
- new net: C27.1, U7.73 (VCAP)
- new net: R27.2, U9.3 (OUT)
- new net: D13.4, R23.2
- new net: D13.2, R25.2
- new net: D13.3, R24.2
- new net +3.3V: C28.1, C29.1, C30.1, C31.1, C32.1, C33.1, C34.1, C35.1, C37.1, FB7.1, R26.1, R30.1, SW1.2, U7.100 (VDD), U7.11 (VDD), U7.21 (VDDA), U7.27 (VDD), U7.50 (VDD), U7.6 (VBAT), U7.75 (VDD), U9.1 (EN), U9.4 (VDD)
- new net BOOT: R29.1, SW1.1, U7.94 (BOOT0)
- new net BUSY_MCU: U7.51 (PB12)
- new net GND: C25.2, C26.2, C27.2, C28.2, C29.2, C30.2, C31.2, C32.2, C33.2, C34.2, C35.2, C36.2, C37.2, D13.1, J7.4, J8.5 (GND), J8.6 (Shield), Q1.2 (S), R28.2, R29.2, R32.2, TP10.1, U7.10 (VSS), U7.19 (VSSA), U7.26 (VSS), U7.49 (VSS), U7.74 (VSS), U7.99 (VSS), U8.2, U8.5, U9.2 (GND)
- new net LED_B: R23.1, U7.63 (PC6)
- new net LED_G: R24.1, U7.64 (PC7)
- new net LED_R: R25.1, U7.65 (PC8)
- new net MISO0_MCU: U7.30 (PA6)
- new net MOSI_MCU: U7.31 (PA7)
- new net Manual_Trigger: U7.57 (PD10)
- new net NRST: C36.1, J7.1, R26.2, U7.14 (NRST)
- new net PA13: J7.2, U7.72 (PA13(JTMS)
- new net PA14: J7.3, U7.76 (PA14(JTCK)
- new net PD1: Q1.1 (G), R32.1, U7.82 (PD1)
- new net PH0: R27.1, U7.12 (PH0)
- new net SCK_MCU: U7.29 (PA5)
- new net Trig_Detect: U7.88 (PD7)
- new net Trig_Enable: U7.62 (PD15)
- new net UART4_CTS: TP9.1, U7.54 (PB15)
- new net UART4_RX: TP7.1, U7.95 (PB8)
- new net UART4_TX: TP8.1, U7.96 (PB9)
- new net USB_D+: J8.3 (D+), U7.71 (PA12), U8.3
- new net USB_D-: J8.2 (D-), U7.70 (PA11), U8.4
- new net USB_ID: J8.4 (ID), U8.1
- new net USB_VBUS: R28.1, R31.2, U7.68 (PA9), U8.6
- new net /CS_MCU: U7.32 (PC4)
- new net /RESET_MCU: Q1.3 (D), R30.2
- no-connect marks 0 -> 61
Other:
- note added: "12MHz_OSC"
- note added: "Crystal Oscillator"
- note added: "Decoupling capacitors"
- note added: "MCU BOOT"
- note added: "NRST Pull-up resistor"
- note added: "RGB LED indecator"
- note added: "Resetting the ADC"
- note added: "STM 32 Programmer"
- note added: "TVS Clamp Array"
- note added: "UART for Debugging"
- note added: "USB"
Changed lines of the file:
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@@
 		(company "N-Well Labs\n\n")
 	)
-)
