File: Power_Management_sch.kicad_sch (KiCad schematic)
At the start: 51 parts, among them J6 Conn_01x03_Pin, U1 LT3093IDD-PBF, U2 LT1763CS8-1.8-TRPBF, U3 LT1763CS8#PBF, U4 LT1763CS8#PBF, U5 LT3042IDD-PBF, U6 LTC6655LNBHMS8-5#PBF

Commit message: edited Power management schematic
Parts:
- removed C19: 1uF, Capacitor_SMD:C_0603_1608Metric, symbol Device:C
- removed D7: Green, LED_SMD:LED_0603_1608Metric, symbol Device:LED
- removed J6: Conn_01x03_Pin, Connector_Phoenix_MC:PhoenixContact_MC_1,5_3-G-3.5_1x03_P3.50mm_Horizontal, symbol Connector:Conn_01x03_Pin
- removed TP1: -5.4, TestPoint:TestPoint_Pad_1.0x1.0mm, symbol focus-symbols:TestPoint
- removed TP2: +1.8V, TestPoint:TestPoint_Pad_1.0x1.0mm, symbol focus-symbols:TestPoint
- removed TP5: +3.3V, TestPoint:TestPoint_Pad_1.0x1.0mm, symbol focus-symbols:TestPoint
- removed TP6: 5V, TestPoint:TestPoint_Pad_1.0x1.0mm, symbol focus-symbols:TestPoint
- removed TP7: +5.4V, TestPoint:TestPoint_Pad_1.0x1.0mm, symbol focus-symbols:TestPoint
- removed TP9: +5V, TestPoint:TestPoint_Pad_1.0x1.0mm, symbol focus-symbols:TestPoint
- added C10, C16, C17, C7, C8: 1uF, Capacitor_SMD:C_0603_1608Metric, symbol Device:C
- added C9: 10uF 25V 1206, Capacitor_SMD:C_1206_3216Metric, symbol Device:C
- added D1: Green, LED_SMD:LED_0603_1608Metric, symbol Device:LED
- added FB1, FB2, FB3, FB4, FB5: 33R, Inductor_SMD:L_0603_1608Metric_Pad1.05x0.95mm_HandSolder, symbol Device:FerriteBead
- added J1: Conn_01x03_Pin, Connector_Phoenix_MC:PhoenixContact_MC_1,5_3-G-3.5_1x03_P3.50mm_Horizontal, symbol Connector:Conn_01x03_Pin
- added TP1: 5.4V, TestPoint:TestPoint_Pad_1.0x1.0mm, symbol majed-symbols:TestPoint
- added TP2: 3.3V, TestPoint:TestPoint_Pad_1.0x1.0mm, symbol majed-symbols:TestPoint
- added TP3: -5.4, TestPoint:TestPoint_Pad_1.0x1.0mm, symbol majed-symbols:TestPoint
- added TP4: 1,,8V, TestPoint:TestPoint_Pad_1.0x1.0mm, symbol majed-symbols:TestPoint
- added TP5, TP6: 5V, TestPoint:TestPoint_Pad_1.0x1.0mm, symbol majed-symbols:TestPoint
- U1: renamed from U3; footprint focus-footprints:SO-8_S_LIT-L -> Majed-footprints:SO-8_S_LIT-L
- U2: renamed from U4; footprint focus-footprints:SO-8_S_LIT-L -> Majed-footprints:SO-8_S_LIT-L
- U4: renamed from U2; footprint focus-footprints:SO-8_S_LIT -> Majed-footprints:SO-8_S_LIT
- U5: renamed from U6; footprint focus-footprints:MSOP-8_MS_LIT-L -> Majed-footprints:MSOP-8_MS_LIT-L
- U6: renamed from U5; footprint focus-footprints:DFN-10_DD_LIT -> Majed-footprints:DFN-10_DD_LIT
- renumbered C26 to C1, C3 to C11, C4 to C12, C1 to C13, C5 to C14, C6 to C15, C20 to C18, C7 to C19, C25 to C2, C23 to C20, C27 to C21, C8 to C22, C2 to C3, C11 to C4, C24 to C5, C12 to C6, D4 to D2, D1 to D3, D2 to D4, D9 to D5, R2 to R1, R13 to R11, R1 to R12, R5 to R13, R22 to R14, R4 to R2, R6 to R3, R7 to R4, R8 to R5, R12 to R6, R3 to R7, R11 to R8, U1 to U3
Connections:
- net +1.8V: now also TP4.1
- net +3.3V: now also TP2.1
- net +5.4V: now also TP1.1
- net +5V: now also TP5.1
- net +6V: now also FB6.2, C7.1, FB1.2, FB2.2, FB3.1, FB5.2, J1.1 (Pin_1); no longer FB6.1
- net -5.4V: now also TP3.1
- net -6V: now also FB4.2, J1.3 (Pin_3)
- net GND: now also C10.2, C16.2, C17.2, C7.2, C8.2, C9.2, D1.1 (K), J1.2 (Pin_2)
- net REF_5V: now also TP6.1
- net at U6.1 (IN), U6.2 (IN), U6.3 (EN/UV)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: now also C16.1, FB5.1
- net at U2.5 (*SHDN), U2.8 (IN): now also C8.1, FB2.1
- net at U3.1 (IN), U3.13 (IN), U3.2 (IN)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: now also C9.1, FB4.1
- net at U1.5 (*SHDN), U1.8 (IN): now also FB1.1
- net at U5.1 (*SHDN), U5.2 (VIN): now also FB6.1, C17.1
- net at R1.2: now also D1.2 (A)
- net at U4.5 (*SHDN), U4.8 (IN): now also C10.1, FB3.2
Other:
- moved on the sheet: C1, C11, C13, C2, C20, C21, C5, D3, D5, R1, R10, R12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

Commit message: All done, Gerberd out :)
Parts:
- added C11, C13: 100uF, Capacitor_Tantalum_SMD:CP_EIA-3528-21_Kemet-B, symbol majed-symbols:C
- added D10: ESD9B5.0ST5G, Diode_SMD:D_SOD-923, symbol majed-symbols:ESD9B5.0ST5G
- added D7: ESD9B3.3ST5G, Diode_SMD:D_SOD-923, symbol majed-symbols:ESD9B3.3ST5G
- C1, C10, C2, C3, C4, C5, C6, C7, C8, C9: symbol Device:C -> majed-symbols:C
- C12: renamed from C11; symbol Device:C -> majed-symbols:C
- C14: renamed from C12; symbol Device:C -> majed-symbols:C
- C15: renamed from C13; symbol Device:C -> majed-symbols:C
- C16: renamed from C14; symbol Device:C -> majed-symbols:C
- C17: renamed from C15; symbol Device:C -> majed-symbols:C
- C18: renamed from C16; symbol Device:C -> majed-symbols:C
- C19: renamed from C17; symbol Device:C -> majed-symbols:C
- C20: renamed from C18; symbol Device:C -> majed-symbols:C
- C21: renamed from C19; symbol Device:C -> majed-symbols:C
- C22: renamed from C20; symbol Device:C -> majed-symbols:C
- C23: renamed from C21; symbol Device:C -> majed-symbols:C
- C24: renamed from C22; symbol Device:C -> majed-symbols:C
- D11: renamed from D5; symbol Device:LED -> majed-symbols:LED
- D12: renamed from D6; symbol Device:LED -> majed-symbols:LED
- D5: renamed from D1; symbol Device:LED -> majed-symbols:LED
- D6: renamed from D2; symbol Device:LED -> majed-symbols:LED
- D8: renamed from D3; symbol Device:LED -> majed-symbols:LED
- D9: renamed from D4; symbol Device:LED -> majed-symbols:LED
- FB1, FB2, FB3, FB4, FB5, FB6: symbol Device:FerriteBead -> majed-symbols:FerriteBead
- J6: renamed from J1; symbol Connector:Conn_01x03_Pin -> majed-symbols:Conn_01x03_Pin
- R10: renamed from R2; symbol Device:R_Small_US -> majed-symbols:R_Small_US
- R11: renamed from R3; symbol Device:R_US -> majed-symbols:R_US
- R12: renamed from R4; symbol Device:R_US -> majed-symbols:R_US
- R13: renamed from R5; symbol Device:R_US -> majed-symbols:R_US
- R14: renamed from R6; symbol Device:R_US -> majed-symbols:R_US
- R15: renamed from R7; symbol Device:R_US -> majed-symbols:R_US
- R16: renamed from R8; symbol Device:R_US -> majed-symbols:R_US
- R17: renamed from R9; symbol Device:R_US -> majed-symbols:R_US
- R18: renamed from R10; symbol Device:R_Small_US -> majed-symbols:R_Small_US
- R19: renamed from R11; symbol Device:R_Small_US -> majed-symbols:R_Small_US
- R20: renamed from R12; symbol Device:R_US -> majed-symbols:R_US
- R21: renamed from R13; symbol Device:R_Small_US -> majed-symbols:R_Small_US
- R22: renamed from R14; symbol Device:R_Small_US -> majed-symbols:R_Small_US
- R9: renamed from R1; symbol Device:R_Small_US -> majed-symbols:R_Small_US
- TP1: value 5.4V -> +5.4V
Connections:
- net +3.3V: now also D7.1 (A1)
- net +6V: now also J6.2 (Pin_2), C13.1; no longer C7.1, J6.1 (Pin_1)
- net -6V: now also C11.1
- net GND: now also J6.1 (Pin_1), C11.2, C13.2, D10.2 (A2), D7.2 (A2); no longer J6.2 (Pin_2)
- net REF_5V: now also D10.1 (A1)
- net at FB1.1, U1.5 (*SHDN), U1.8 (IN): now also C7.1
Other:
- moved on the sheet: C7, D12, FB1, R22, TP6
