File: ADC_Driver_Stage-Final-Buffer.kicad_sch (KiCad schematic)
At the start: 0 parts

Commit message: All done, Gerberd out :)
Parts:
- added C43, C44, C45, C46: 0.01uF 0603, Capacitor_SMD:C_0603_1608Metric, symbol majed-symbols:C
- added C47, C48: 10uF 25V 1206, Capacitor_SMD:C_1206_3216Metric, symbol majed-symbols:C
- added C49, C50: 1000pF, Capacitor_SMD:C_0603_1608Metric, symbol majed-symbols:C
- added FB8, FB9: 33R, Inductor_SMD:L_0603_1608Metric_Pad1.05x0.95mm_HandSolder, symbol majed-symbols:FerriteBead
- added R36, R37: 10, Resistor_SMD:R_0805_2012Metric, symbol majed-symbols:R_US
- added R38, R39: 33, Resistor_SMD:R_0603_1608Metric, symbol majed-symbols:R_US
- added U11: ADA4896-2ARMZ, Majed-footprints:RM_8_ADI, symbol majed-symbols:ADA4896-u_1
Connections:
- new net: C43.1, R37.1, U11.5 (+IN2)
- new net: R39.2, U11.6 (-IN2), U11.7 (OUT2)
- new net: C44.1, C47.1, FB8.2, U11.8 (+VS)
- new net: C46.1, C48.1, FB9.2, U11.4 (-VS)
- new net: C45.1, R36.2, U11.3 (+IN1)
- new net: R38.2, U11.1 (OUT1), U11.2 (-IN1)
- new net +5.4V: FB8.1
- new net -5.4V: FB9.1
- new net External_IN+: R36.1
- new net External_IN-: R37.2
- new net Filtered_IN+: C49.1, R38.1
- new net Filtered_IN-: C50.1, R39.1
- new net GND: C43.2, C44.2, C45.2, C46.2, C47.2, C48.2, C49.2, C50.2
Other:
- note added: "Signal Conditioning & Buffering [ IN + ]"
- note added: "Signal Conditioning & Buffering [ IN - ]"

Commit message: Extra signal conditioning
Parts:
- removed FB8, FB9: 33R, Inductor_SMD:L_0603_1608Metric_Pad1.05x0.95mm_HandSolder, symbol majed-symbols:FerriteBead
- added R74, R76: 33, Resistor_SMD:R_0603_1608Metric, symbol majed-symbols:R_US
Connections:
- net +5.4V: now also R74.2
- net -5.4V: now also R76.2
- net at C44.1, C47.1, U11.8 (+VS): now also R74.1
- net at C46.1, C48.1, U11.4 (-VS): now also R76.1
Changed lines of the file:
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@@
+	)
+	(symbol
+		(lib_id "majed-symbols:R_US")
+		(at 48.26 92.71 270)
+		(unit 1)
+		(exclude_from_sim no)
+		(in_bom yes)
+		(on_board yes)
+		(dnp no)
+		(fields_autoplaced yes)
+		(property "Reference" "R76"
+			(at 48.26 86.36 90)
+			(effects
+				(font
+					(size 1.27 1.27)
+				)
+			)
+		)
+		(property "Value" "33"
+			(at 48.26 88.9 90)
+			(effects
+				(font
+					(size 1.27 1.27)
+				)
+			)
+		)
+		(property "Footprint" "Resistor_SMD:R_0603_1608Metric"
+			(at 48.006 93.726 90)
+			(effects
+				(font
+					(size 1.27 1.27)
+				)
+				(hide yes)
+			)
+		)
+		(property "Datasheet" "~"
+			(at 48.26 92.71 0)
+			(effects
+				(font
+					(size 1.27 1.27)
+				)
+				(hide yes)
+			)
+		)
+		(property "Description" "Resistor, US symbol"
+			(at 48.26 92.71 0)
+			(effects
+				(font
+					(size 1.27 1.27)
+				)
+				(hide yes)
+			)
+		)
+		(property "Manufacturer" "YAGEO"
+			(at 48.26 92.71 0)
+			(effects
+				(font
+					(size 1.27 1.27)
+				)
+				(hide yes)
+			)
+		)
+		(property "Digikey" "311-33GRCT-ND"
+			(at 48.26 92.71 0)
+			(effects
+				(font
+					(size 1.27 1.27)
+				)
+				(hide yes)
+			)
+		)
+		(property "Mfg part #" "RC0603FR-072KL"
+			(at 48.26 92.71 0)
+			(effects
+				(font
+					(size 1.27 1.27)
+				)
+				(hide yes)
+			)
+		)
+		(pin "2"
+		)
+		(pin "1"
+		)
+		(instances
+			(project "NanoPulse"
+				(path "/86831492-4864-4889-ae52-8b89506c40dd/8f0d12f0-b179-4281-8c43-e729f8a20598"
+					(reference "R76")
+					(unit 1)
+				)
+				(path "/86831492-4864-4889-ae52-8b89506c40dd/dab339a6-33d6-4321-af03-924f4dc6f0cd"
+					(reference "R77")
+					(unit 1)
+				)
+			)
+		)
 	)
 	(symbol
@@
 	)
 	(symbol
-		(lib_id "majed-symbols:FerriteBead")
-		(at 48.26 92.71 90)
-		(unit 1)
-		(exclude_from_sim no)
-		(in_bom yes)
-		(on_board yes)
-		(dnp no)
-		(property "Reference" "FB9"
-			(at 50.546 86.106 90)
-			(effects
-				(font
-					(size 1.27 1.27)
-				)
-			)
-		)
-		(property "Value" "33R"
-			(at 50.546 88.646 90)
-			(effects
-				(font
-					(size 1.27 1.27)
-				)
-			)
-		)
-		(property "Footprint" "Inductor_SMD:L_0603_1608Metric_Pad1.05x0.95mm_HandSolder"
-			(at 48.26 94.488 90)
-			(effects
-				(font
-					(size 1.27 1.27)
-				)
-				(hide yes)
-			)
-		)
-		(property "Datasheet" "~"
-			(at 48.26 92.71 0)
-			(effects
-				(font
-					(size 1.27 1.27)
-				)
-				(hide yes)
-			)
-		)
-		(property "Description" "Ferrite bead"
-			(at 48.26 92.71 0)
-			(effects
-				(font
-					(size 1.27 1.27)
-				)
-				(hide yes)
-			)
-		)
-		(property "Manufacturer" "Murata Electronics "
-			(at 48.26 92.71 0)
-			(effects
-				(font
-					(size 1.27 1.27)
-				)
-				(hide yes)
-			)
-		)
-		(property "Digikey" "490-5220-1-ND"
-			(at 48.26 92.71 0)
-			(effects
-				(font
-					(size 1.27 1.27)
-				)
-				(hide yes)
-			)
-		)
-		(property "Mfg part #" "BLM18PG330SN1D"
-			(at 48.26 92.71 0)
-			(effects
-				(font
-					(size 1.27 1.27)
-				)
-				(hide yes)
-			)
-		)
-		(pin "1"
-		)
-		(pin "2"
-		)
-		(instances
-			(project "NanoPulse"
-				(path "/86831492-4864-4889-ae52-8b89506c40dd/8f0d12f0-b179-4281-8c43-e729f8a20598"
-					(reference "FB9")
-					(unit 1)
-				)
-				(path "/86831492-4864-4889-ae52-8b89506c40dd/dab339a6-33d6-4321-af03-924f4dc6f0cd"
-					(reference "FB11")
-					(unit 1)
-				)
-			)
-		)
-	)
-	(symbol
 		(lib_id "majed-symbols:R_US")
 		(at 49.53 146.05 270)
@@
 	)
 	(symbol
+		(lib_id "majed-symbols:R_US")
+		(at 48.26 35.56 270)
+		(unit 1)
+		(exclude_from_sim no)
+		(in_bom yes)
+		(on_board yes)
+		(dnp no)
+		(fields_autoplaced yes)
+		(property "Reference" "R74"
+			(at 48.26 29.21 90)
+			(effects
+				(font
+					(size 1.27 1.27)
+				)
+			)
+		)
+		(property "Value" "33"
+			(at 48.26 31.75 90)
+			(effects
+				(font
+					(size 1.27 1.27)
+				)
+			)
+		)
+		(property "Footprint" "Resistor_SMD:R_0603_1608Metric"
+			(at 48.006 36.576 90)
+			(effects
+				(font
+					(size 1.27 1.27)
+				)
+				(hide yes)
+			)
+		)
+		(property "Datasheet" "~"
+			(at 48.26 35.56 0)
+			(effects
+				(font
+					(size 1.27 1.27)
+				)
+				(hide yes)
+			)
+		)
+		(property "Description" "Resistor, US symbol"
+			(at 48.26 35.56 0)
+			(effects
+				(font
+					(size 1.27 1.27)
+				)
+				(hide yes)
+			)
+		)
+		(property "Manufacturer" "YAGEO"
+			(at 48.26 35.56 0)
+			(effects
+				(font
+					(size 1.27 1.27)
+				)
+				(hide yes)
+			)
+		)
+		(property "Digikey" "311-33GRCT-ND"
+			(at 48.26 35.56 0)
+			(effects
+				(font
+					(size 1.27 1.27)
+				)
+				(hide yes)
+			)
+		)
+		(property "Mfg part #" "RC0603FR-072KL"
+			(at 48.26 35.56 0)
+			(effects
+				(font
+					(size 1.27 1.27)
+				)
+				(hide yes)
+			)
+		)
+		(pin "2"
+		)
+		(pin "1"
+		)
+		(instances
+			(project "NanoPulse"
+				(path "/86831492-4864-4889-ae52-8b89506c40dd/8f0d12f0-b179-4281-8c43-e729f8a20598"
+					(reference "R74")
+					(unit 1)
+				)
+				(path "/86831492-4864-4889-ae52-8b89506c40dd/dab339a6-33d6-4321-af03-924f4dc6f0cd"
+					(reference "R75")
+					(unit 1)
+				)
+			)
+		)
+	)
+	(symbol
 		(lib_id "majed-symbols:C")
 		(at 140.97 152.4 0)
@@
 					(unit 1)
 				)
-			)
-		)
-	)
-	(symbol
-		(lib_id "majed-symbols:FerriteBead")
-		(at 48.26 35.56 90)
-		(unit 1)
-		(exclude_from_sim no)
-		(in_bom yes)
-		(on_board yes)
-		(dnp no)
-		(property "Reference" "FB8"
-			(at 50.546 28.956 90)
-			(effects
-				(font
-					(size 1.27 1.27)
-				)
-			)
-		)
-		(property "Value" "33R"
-			(at 50.8 31.496 90)
-			(effects
-				(font
-					(size 1.27 1.27)
-				)
-			)
-		)
-		(property "Footprint" "Inductor_SMD:L_0603_1608Metric_Pad1.05x0.95mm_HandSolder"
-			(at 48.26 37.338 90)
-			(effects
-				(font
-					(size 1.27 1.27)
-				)
-				(hide yes)
-			)
-		)
-		(property "Datasheet" "~"
-			(at 48.26 35.56 0)
-			(effects
-				(font
-					(size 1.27 1.27)
-				)
-				(hide yes)
-			)
-		)
-		(property "Description" "Ferrite bead"
-			(at 48.26 35.56 0)
-			(effects
-				(font
-					(size 1.27 1.27)
-				)
-				(hide yes)
-			)
-		)
-		(property "Manufacturer" "Murata Electronics "
-			(at 48.26 35.56 0)
-			(effects
-				(font
-					(size 1.27 1.27)
-				)
-				(hide yes)
-			)
-		)
-		(property "Digikey" "490-5220-1-ND"
-			(at 48.26 35.56 0)
-			(effects
-				(font
-					(size 1.27 1.27)
-				)
-				(hide yes)
-			)
-		)
-		(property "Mfg part #" "BLM18PG330SN1D"
-			(at 48.26 35.56 0)
-			(effects
-				(font
-					(size 1.27 1.27)
-				)
-				(hide yes)
-			)
-		)
-		(pin "1"
-		)
-		(pin "2"
-		)
-		(instances
-			(project "NanoPulse"
-				(path "/86831492-4864-4889-ae52-8b89506c40dd/8f0d12f0-b179-4281-8c43-e729f8a20598"
-					(reference "FB8")
-					(unit 1)
-				)
-				(path "/86831492-4864-4889-ae52-8b89506c40dd/dab339a6-33d6-4321-af03-924f4dc6f0cd"
-					(reference "FB10")
-					(unit 1)
-				)
