File: NanoPulse.kicad_pcb (KiCad board)
At the start: 4 copper layers, 113 x 61.6 mm, 240 parts, among them J1 SMA_conn, J2 SMA_conn, J3 SMA_conn, J4 SMA_conn, J5 SMA_conn, J6 Conn_01x03_Pin, J7 STM32 PROGRAMER, J8 USB_B_Micro, Q1 2N7002K, SW1 Push - BOOT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

Commit message: Extra signal conditioning
Parts:
- removed FB10, FB11, FB8, FB9: 33R, Inductor_SMD:L_0603_1608Metric_Pad1.05x0.95mm_HandSolder
- added R73: 33, Resistor_SMD:R_0603_1608Metric, B.Cu at (161.9, 85.9)
- added R74: 33, Resistor_SMD:R_0603_1608Metric, B.Cu at (104.8, 73.7)
- added R75: 33, Resistor_SMD:R_0603_1608Metric, B.Cu at (178.4, 83.2)
- added R76: 33, Resistor_SMD:R_0603_1608Metric, B.Cu at (128.3, 80.7)
- added R77: 33, Resistor_SMD:R_0603_1608Metric, B.Cu at (156.5, 76.4)
- added TP20: CNV_EXT_RAW, TestPoint:TestPoint_Pad_1.0x1.0mm, F.Cu at (174.0, 108.6)
- added TP21: CNV_3V3_OUT, TestPoint:TestPoint_Pad_1.0x1.0mm, B.Cu at (158.3, 99.5)
- added TP22: CNV_1V8_ADC, TestPoint:TestPoint_Pad_1.0x1.0mm, B.Cu at (171.8, 90.3)
- R72: value 500 -> 33
Connections:
- net /Trigger Circuit/Trigger_Signal renamed /Trigger Circuit/CNV_EXT_RAW
- net Net-(U19-Pad4) renamed /Trigger Circuit/CNV_GATED_3V3
- U15 pad 9: CNV -> Net-(U15-A6)
Routing:
- net Net-(U15-A6): track 0.00 -> 8.08 mm, vias 0 -> 2
- net CNV: track 44.9 -> 52.8 mm, vias 3 -> 1
- net /Trigger Circuit/CNV_EXT_RAW: track 15.0 -> 20.3 mm
- net CNV_3.3: track 11.7 -> 13.4 mm
- net REF_5V: track 131.3 -> 132.1 mm
