File: Single_To_Diff_Driver_Stage.kicad_sch (KiCad schematic)
At the start: 0 parts

Commit message: All done, Gerberd out :)
Parts:
- added C59, C60: 0.01uF 0603, Capacitor_SMD:C_0603_1608Metric, symbol majed-symbols:C
- added C61: 0.1uF, Capacitor_SMD:C_0603_1608Metric, symbol majed-symbols:C
- added C62, C63: 2700pF, Capacitor_SMD:C_0805_2012Metric, symbol majed-symbols:C
- added C64, C65: 1000pF, Capacitor_SMD:C_0603_1608Metric, symbol majed-symbols:C
- added C66, C67: 1uF, Capacitor_SMD:C_0603_1608Metric, symbol majed-symbols:C
- added FB12, FB13: 33R, Inductor_SMD:L_0603_1608Metric_Pad1.05x0.95mm_HandSolder, symbol majed-symbols:FerriteBead
- added R44, R45: DNI, Resistor_SMD:R_0603_1608Metric, symbol majed-symbols:R_Small_US
- added R46, R48: 10K, Resistor_SMD:R_0603_1608Metric, symbol majed-symbols:R_Small_US
- added R47, R49: 54.09, Resistor_SMD:R_0603_1608Metric, symbol majed-symbols:R_Small_US
- added R50, R51: 1K, Resistor_SMD:R_0603_1608Metric, symbol majed-symbols:R_Small_US
- added R52, R53: 2K, Resistor_SMD:R_0603_1608Metric, symbol majed-symbols:R_Small_US
- added R54, R55: DNI, Resistor_SMD:R_0603_1608Metric, symbol majed-symbols:R_US
- added U13: ADA4945, Majed-footprints:LFCSP16_ADA4945-1ACPZ-R2_ADI-L, symbol majed-symbols:ADA4945
Connections:
- new net: C66.1, FB12.1, U13.12 (~{DISABLE1}), U13.5 (MODE), U13.6 (+VS), U13.7 (+VS), U13.8 (+VCLAMP)
- new net: R55.1, U13.10 (+OUT)
- new net: C63.2, R51.1, R53.1, U13.2 (+IN1)
- new net: C63.1, R53.2, U13.1 (-FB)
- new net: C61.2, R46.2, R48.1, U13.9 (VOCM)
- new net: C62.1, R50.1, R52.2, U13.3 (-IN1)
- new net: C62.2, R52.1, U13.4 (+FB)
- new net: R54.1, U13.11 (-OUT)
- new net: C59.1, R45.1, R47.1, R50.2
- new net: C67.1, FB13.1, U13.13 (-VCLAMP), U13.14 (-VS), U13.15 (-VS), U13.16 (DGND), U13.17 (-VS)
- new net: C60.1, R44.1, R49.1, R51.2
- new net +5.4V: FB12.2
- new net -5.4V: FB13.2
- new net GND: C59.2, C60.2, C61.1, C64.2, C65.2, C66.2, C67.2, R47.2, R48.2, R49.2
- new net REF_5V: R46.1
- new net S_External_IN+: R44.2
- new net S_External_IN-: R45.2
- new net S_Filtered_IN+: C65.1, R55.2
- new net S_Filtered_IN-: C64.1, R54.2
Other:
- note added: "Power Conditioning for Op-Amp"
- note added: "Signal Conditioning & ADC Driver [ Single to Diff ]"

Commit message: Extra signal conditioning
Other:
- moved on the sheet: R46
Changed lines of the file:
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@@
-	)
-	(junction
-		(at 59.69 92.71)
-		(diameter 0)
-		(color 0 0 0 0)
 	)
 	(junction
@@
 	(wire
 		(pts
-			(xy 59.69 85.09) (xy 59.69 81.28)
+			(xy 64.77 85.09) (xy 64.77 81.28)
 		)
 		(stroke
@@
 	(wire
 		(pts
-			(xy 59.69 81.28) (xy 55.88 81.28)
+			(xy 64.77 81.28) (xy 60.96 81.28)
 		)
 		(stroke
@@
 	(wire
 		(pts
-			(xy 64.77 92.71) (xy 59.69 92.71)
-		)
-		(stroke
-			(width 0.635)
-			(type default)
-		)
-	)
-	(wire
-		(pts
 			(xy 64.77 57.15) (xy 64.77 55.88)
 		)
@@
 	(wire
 		(pts
-			(xy 59.69 90.17) (xy 59.69 92.71)
+			(xy 64.77 90.17) (xy 64.77 92.71)
 		)
 		(stroke
@@
 	(wire
 		(pts
-			(xy 59.69 92.71) (xy 53.34 92.71)
+			(xy 53.34 92.71) (xy 64.77 92.71)
 		)
 		(stroke
@@
 	(global_label "REF_5V"
 		(shape input)
-		(at 55.88 81.28 180)
+		(at 60.96 81.28 180)
 		(fields_autoplaced yes)
 		(effects
@@
 		)
 		(property "Intersheetrefs" "${INTERSHEET_REFS}"
-			(at 45.6455 81.28 0)
+			(at 50.7255 81.28 0)
 			(effects
 				(font
@@
 		)
 		(property "Dsc" "VAMP+"
-			(at 55.88 83.566 0)
+			(at 60.96 83.566 0)
 			(effects
 				(font
@@
 	(symbol
 		(lib_id "majed-symbols:R_Small_US")
-		(at 59.69 87.63 0)
+		(at 64.77 87.63 0)
 		(mirror y)
 		(unit 1)
@@
 		(dnp no)
 		(property "Reference" "R46"
-			(at 63.5 89.027 0)
+			(at 68.58 89.027 0)
 			(effects
 				(font
@@
 		)
 		(property "Value" "10K"
-			(at 63.5 86.7156 0)
+			(at 68.58 86.7156 0)
 			(effects
 				(font
@@
 		)
 		(property "Footprint" "Resistor_SMD:R_0603_1608Metric"
-			(at 59.69 87.63 0)
+			(at 64.77 87.63 0)
 			(effects
 				(font
@@
 		)
 		(property "Datasheet" "~"
-			(at 59.69 87.63 0)
+			(at 64.77 87.63 0)
 			(effects
 				(font
@@
 		)
 		(property "Description" "Resistor, small US symbol"
-			(at 59.69 87.63 0)
+			(at 64.77 87.63 0)
 			(effects
 				(font
@@
 		)
 		(property "Manufacturer" "YAGEO"
-			(at 59.69 87.63 0)
+			(at 64.77 87.63 0)
 			(effects
 				(font
@@
 		)
 		(property "Digikey" "311-10.0KHRCT-ND"
-			(at 59.69 87.63 0)
+			(at 64.77 87.63 0)
 			(effects
 				(font
@@
 		)
 		(property "Mfg part #" "RC0603FR-0710KL"
-			(at 59.69 87.63 0)
-			(effects
-				(font
+			(at 64.77 87.63 0)
+			(effects
+				(font
