File: Trigger_Circuit.kicad_sch (KiCad schematic)
At the start: 0 parts

Commit message: All done, Gerberd out :)
Parts:
- added C83, C84, C85: 0.1uF, Capacitor_SMD:C_0603_1608Metric, symbol majed-symbols:C_Small
- added R71: 50 (1210), Resistor_SMD:R_1210_3225Metric_Pad1.30x2.65mm_HandSolder, symbol majed-symbols:R_US
- added R72: 500, Resistor_SMD:R_0603_1608Metric, symbol majed-symbols:R_US
- added TP17: Trig_Detect, TestPoint:TestPoint_Pad_1.0x1.0mm, symbol majed-symbols:TestPoint
- added TP18: Trig_Enable, TestPoint:TestPoint_Pad_1.0x1.0mm, symbol majed-symbols:TestPoint
- added TP19: Manual_Trigger, TestPoint:TestPoint_Pad_1.0x1.0mm, symbol majed-symbols:TestPoint
- added U18: 74LVC2G17GW,125, Package_TO_SOT_SMD:SOT-363_SC-70-6, symbol majed-symbols:74LVC2G17
- added U19: 74AHC1G08GW,125, Package_TO_SOT_SMD:SOT-353_SC-70-5, symbol majed-symbols:74AHC1G08
- added U20: 74AHC1G32GW,125, Package_TO_SOT_SMD:SOT-353_SC-70-5, symbol majed-symbols:74AHC1G32
Connections:
- new net: U19.4, U20.2
- new net: R72.1, U18.1
- new net +3.3V: C83.1, C84.1, C85.1, U18.5 (VCC), U19.5 (VCC), U20.5 (VCC)
- new net CNV_3.3: U20.4
- new net GND: C83.2, C84.2, C85.2, R71.2, U18.2 (GND), U18.3, U19.3 (GND), U20.3 (GND)
- new net Manual_Trigger: TP19.1, U20.1
- new net Trig_Detect: TP17.1, U18.6, U19.2
- new net Trig_Enable: TP18.1, U19.1
- new net Trigger_Signal: R71.1, R72.2
- no-connect marks 0 -> 1
Other:
- note added: "Trigger Circuit"

Commit message: Extra signal conditioning
Parts:
- added TP20: CNV_EXT_RAW, TestPoint:TestPoint_Pad_1.0x1.0mm, symbol majed-symbols:TestPoint
- added TP21: CNV_3V3_OUT, TestPoint:TestPoint_Pad_1.0x1.0mm, symbol majed-symbols:TestPoint
- R72: value 500 -> 33; Digikey 13-RT0603BRC07500RLCT-ND -> 311-33GRCT-ND; Mfg part # RT0603BRC07500RL -> RC0603FR-072KL
Connections:
- net CNV_3.3: now also TP21.1
- net CNV_GATED_3V3: now reaches U19.4, U20.2
- net Trigger_Signal renamed CNV_EXT_RAW
- net CNV_EXT_RAW: now also TP20.1
Other:
- note added: "Populate R71 only when using external 50 Ω trigger"
