File: Voltage_Translator.kicad_sch (KiCad schematic)
At the start: 0 parts

Commit message: All done, Gerberd out :)
Parts:
- added C77, C78, C79, C80, C81, C82: 0.1uF, Capacitor_SMD:C_0603_1608Metric, symbol majed-symbols:C
- added R68, R69, R70: 33, Resistor_SMD:R_0603_1608Metric, symbol majed-symbols:R_US
- added U15: FXLH42245MPX, Majed-footprints:MLP24_4P5X3P5_ONS, symbol majed-symbols:FXLH42245MPX_1
- added U16: FXL2T245L10X, Majed-footprints:MICROPAK10_2P1X1P6_ONS-L, symbol majed-symbols:FXL2T245L10X
- added U17: FXLH42245MPX, Majed-footprints:MLP24_4P5X3P5_ONS, symbol majed-symbols:FXLH42245MPX
Connections:
- new net: R69.2, U15.4 (A1)
- new net: R70.2, U15.5 (A2)
- new net: R68.2, U15.3 (A0)
- new net +1.8V: C77.1, C78.1, C81.1, U15.1 (VCCA), U16.1 (VCCA), U16.4 (T/*R), U17.1 (VCCA), U17.2 (T/*R)
- new net +3.3V: C79.1, C80.1, C82.1, U15.23 (VCCB), U15.24 (VCCB), U16.10 (VCCB), U17.23 (VCCB), U17.24 (VCCB)
- new net BUSY: U16.2 (A0)
- new net BUSY_MCU: U16.9 (B0)
- new net CNV: U15.9 (A6)
- new net CNV_3.3: U15.15 (B6)
- new net GND: C77.2, C78.2, C79.2, C80.2, C81.2, C82.2, U15.11 (GND), U15.12 (GND), U15.13 (GND), U15.16 (B5), U15.17 (B4), U15.18 (B3), U15.2 (T/*R), U15.22 (*OE), U15.25 (EPAD), U16.3 (A1), U16.5 (GND), U16.6 (GND), U16.7 (*OE), U17.10 (A7), U17.11 (GND), U17.12 (GND), U17.13 (GND), U17.22 (*OE), U17.25 (EPAD), U17.4 (A1), U17.5 (A2), U17.6 (A3), U17.7 (A4), U17.8 (A5), U17.9 (A6)
- new net MISO0: U17.3 (A0)
- new net MISO0_MCU: U17.21 (B0)
- new net MOSI: R68.1
- new net MOSI_MCU: U15.21 (B0)
- new net SCK: R70.1
- new net SCK_MCU: U15.19 (B2)
- new net /CS: R69.1
- new net /CS_MCU: U15.20 (B1)
- new net /RESET: U15.10 (A7)
- new net /RESET_MCU: U15.14 (B7)
- no-connect marks 0 -> 11
Other:
- note added: "From 1.8V to 3.3V MCU Busy Pin"
- note added: "From 1.8V to 3.3V SPI"
- note added: "From 3.3V to 1.8V ADC"
- note added: "Voltage Level Transilator [ 1.8V - 3.3V ]"
- note added: "Voltage Level Transilator [ BUSY ]"
- note added: "Voltage Level Transilator [ For Octo-SPI ]"

Commit message: Extra signal conditioning
Parts:
- added R73: 33, Resistor_SMD:R_0603_1608Metric, symbol majed-symbols:R_US
- added TP22: CNV_1V8_ADC, TestPoint:TestPoint_Pad_1.0x1.0mm, symbol majed-symbols:TestPoint
Connections:
- net CNV: now also R73.2, TP22.1; no longer U15.9 (A6)
- new net: R73.1, U15.9 (A6)
